Commit message: 1207

File: urdf/camera.urdf.xacro (robot description, xacro)
@@ -1,12 +1,14 @@
 <?xml version="1.0" ?>
-<robot name="camera" xmlns:xacro="http://ros.org/wiki/xacro">
+<robot name="camera" xmlns:xacro="http://www.ros.org/wiki/xacro">
 <xacro:property name="PI" value="3.14159265358979"/>
+<xacro:macro name="camera_macro" params="name parent xyz">
 <!-- Let's try to model camera! -->
 <!-- reference: https://qiita.com/srs/items/7d78f9ad21a0e61f5bff -->
 <!-- gazebo official: http://gazebosim.org/tutorials?tut=ros_gzplugins -->
-    <!-- <link name="camera">
+    <link name="${name}_sensor">
         <visual>
+	    <origin xyz="0 0 0" rpy="0 0 0"/>
             <geometry>
-                <box size="0.01 0.005 0.005"/>
+                <box size="0.005 0.005 0.005"/>
             </geometry>
         </visual>
@@ -17,11 +19,54 @@
                      izx="0" izy="0" izz="0.001" />
         </inertial>
+	<collision>
+	    <origin xyz="0 0 0" rpy="0 0 0"/>
+            <geometry>
+                <box size="0.005 0.005 0.005"/>
+            </geometry>
+        </collision>
     </link>
     <joint name="${name}_sensor_joint" type="fixed">
-        <parent link=""/>
-        <child link=""/>
-        <origin xyz="" rpy=""/>
+	    <axis xyz="0 1 0"/>
+	    <parent link="${parent}"/>
+	    <child link="${name}_sensor"/>
+	    <origin xyz="${xyz}" rpy="${radians(-90)} ${radians(180)} 0"/>
     </joint>
     <gazebo reference="${name}_sensor">
-    </gazebo> -->
+      <sensor type="camera" name="${name}">
+        <update_rate>30.0</update_rate>
+        <camera name="${name}">
+	  <pose>0 0 0 0 ${radians(-90)} ${radians(-90)}</pose>
+	  <horizontal_fov>1.3962634</horizontal_fov>
+	  <image>
+	    <width>800</width>
+	    <height>600</height>
+	    <format>R8G8B8</format>
+	  </image>
+	  <clip>
+	    <near>0.02</near>
+	    <far>300</far>
+	  </clip>
+	  <noise>
+	    <type>gaussian</type>
+	    <mean>0.0</mean>
+	    <stddev>0.007</stddev>
+	  </noise>
+        </camera>
+        <plugin name="camera_controller" filename="libgazebo_ros_camera.so">
+	  <alwaysOn>true</alwaysOn>
+	  <updateRate>0.0</updateRate>
+	  <cameraName>${name}</cameraName>
+	  <imageTopicName>image_raw</imageTopicName>
+	  <cameraInfoTopicName>camera_info</cameraInfoTopicName>
+	  <frameName>${name}_link</frameName>
+	  <hackBaseline>0.07</hackBaseline>
+	  <distortionK1>0.0</distortionK1>
+	  <distortionK2>0.0</distortionK2>
+	  <distortionK3>0.0</distortionK3>
+	  <distortionT1>0.0</distortionT1>
+	  <distortionT2>0.0</distortionT2>
+         </plugin>
+      </sensor>
+    </gazebo>
+  </xacro:macro>
 </robot>

File: urdf/light_sensor.urdf.xacro (robot description, xacro)
@@ -2,5 +2,5 @@
 <!-- p.92  -->
 <robot name="light_sensor" xmlns:xacro="http://ros.org/wiki/xacro">
-<xacro:property name="light_range" value="0.18"/>
+<xacro:property name="light_range" value="1.00"/>
 <xacro:property name="min_range" value="0.01"/>
 <xacro:property name="max_range" value="1.0"/>
@@ -35,5 +35,5 @@
                         <sapmles>10</sapmles>
                         <resolution>1</resolution>
-                        <min_angle>${light_range/2}</min_angle>
+                        <min_angle>-${light_range/2}</min_angle>
                         <max_angle>${light_range/2}</max_angle>
                     </horizontal>

File: urdf/robot.urdf.xacro (robot description, xacro)
@@ -1,4 +1,4 @@
 <?xml version="1.0" ?>
-<robot name="SimpleMouse" xmlns:xacro="http://ros.org/wiki/xacro">
+<robot name="SimpleMouse" xmlns:xacro="http://www.ros.org/wiki/xacro">
  <xacro:include filename="$(find sd_sample_pkg)/urdf/body.urdf.xacro" />
  <xacro:include filename="$(find sd_sample_pkg)/urdf/wheel.urdf.xacro" />
@@ -21,3 +21,4 @@
  <xacro:wheel rl="l" parent="body" />
  <xacro:gazebo_light_sensor name="front" parent="body" xyz="0 0.02 0.03" direction="0" />
+ <xacro:camera_macro name="cfront" parent="body" xyz="0 0 0"/>
 </robot>

Commit message: 0114

File: urdf/camera.urdf.xacro (robot description, xacro)
@@ -2,5 +2,5 @@
 <robot name="camera" xmlns:xacro="http://www.ros.org/wiki/xacro">
 <xacro:property name="PI" value="3.14159265358979"/>
-<xacro:macro name="camera_macro" params="name parent xyz">
+<xacro:macro name="camera_macro" params="name parent xyz rpy">
 <!-- Let's try to model camera! -->
 <!-- reference: https://qiita.com/srs/items/7d78f9ad21a0e61f5bff -->
@@ -30,5 +30,5 @@
 	    <parent link="${parent}"/>
 	    <child link="${name}_sensor"/>
-	    <origin xyz="${xyz}" rpy="${radians(-90)} ${radians(180)} 0"/>
+	    <origin xyz="${xyz}" rpy="${rpy}"/>
     </joint>
     <gazebo reference="${name}_sensor">

File: urdf/light_sensor.urdf.xacro (robot description, xacro)
@@ -2,7 +2,7 @@
 <!-- p.92  -->
 <robot name="light_sensor" xmlns:xacro="http://ros.org/wiki/xacro">
-<xacro:property name="light_range" value="1.00"/>
+<xacro:property name="light_range" value="6"/>
 <xacro:property name="min_range" value="0.01"/>
-<xacro:property name="max_range" value="1.0"/>
+<xacro:property name="max_range" value="0.5"/>
 <xacro:property name="PI" value="3.14159265358979"/>
 <xacro:macro name="gazebo_light_sensor" params="name parent xyz direction">
@@ -35,6 +35,6 @@
                         <sapmles>10</sapmles>
                         <resolution>1</resolution>
-                        <min_angle>-${light_range/2}</min_angle>
-                        <max_angle>${light_range/2}</max_angle>
+			<min_angle>${radians(-180)}</min_angle>
+                        <max_angle>${radians(180)}</max_angle>
                     </horizontal>
                 </scan>

File: urdf/robot.urdf.xacro (robot description, xacro)
@@ -21,4 +21,5 @@
  <xacro:wheel rl="l" parent="body" />
  <xacro:gazebo_light_sensor name="front" parent="body" xyz="0 0.02 0.03" direction="0" />
- <xacro:camera_macro name="cfront" parent="body" xyz="0 0 0"/>
+ <xacro:camera_macro name="camera/rgb" parent="body" xyz="0 0 0" rpy="${radians(-90)} ${radians(180)} 0"/>
+ <!--<xacro:camera_macro name="under" parent="body" xyz="0 -1 0" rpy="0 ${radians(180)} 0"/>-->
 </robot>
